Commit message: Add RGB camera

File: src/armbot_description/urdf/armbot.urdf.xacro (robot description, xacro)
@@ -12,4 +12,10 @@
             </geometry>
         </visual>
+        <collision>
+            <origin rpy="0 0 0" xyz="-0.5 -0.5 0"/>
+            <geometry>
+                <mesh filename="package://armbot_description/meshes/basement.STL" scale="0.01 0.01 0.01"/>
+            </geometry>
+        </collision>
     </link>
     <joint name="virtual_joint" type="fixed">
@@ -25,4 +31,10 @@
             </geometry>
         </visual>
+        <collision>
+            <origin rpy="0 0 0" xyz="-0.39 -0.39 -0.56"/>
+            <geometry>
+                <mesh filename="package://armbot_description/meshes/base_plate.STL" scale="0.01 0.01 0.01"/>
+            </geometry>
+        </collision>
     </link>
     <joint name="joint_1" type="revolute">
@@ -62,4 +74,10 @@
             </geometry>
         </visual>
+        <collision>
+            <origin rpy="${PI / 2} 0 ${PI / 2}" xyz="-0.03 -0.4 -0.06"/>
+            <geometry>
+                <mesh filename="package://armbot_description/meshes/horizontal_arm.STL" scale="0.01 0.01 0.01"/>
+            </geometry>
+        </collision>
     </link>
     <joint name="joint_3" type="revolute">
@@ -78,4 +96,10 @@
             </geometry>
         </visual>
+        <collision>
+            <origin rpy="0 0 ${PI / 2}" xyz="0 -0.05 -0.15"/>
+            <geometry>
+                <mesh filename="package://armbot_description/meshes/claw_support.STL" scale="0.01 0.01 0.01"/>
+            </geometry>
+        </collision>
     </link>
     <joint name ="horizontal_arm_to_claw_support" type="fixed">
@@ -117,3 +141,16 @@
         <mimic joint="joint_4" multiplier="-1"/>
     </joint>
+    <link name="rgb_camera">
+        <visual>
+            <origin rpy="-1.57 0 -1.57" xyz="-0.1 0.125 0.15"/>
+            <geometry>
+                <mesh filename="package://armbot_description/meshes/pi_camera.STL" scale="0.01 0.01 0.01"/>
+            </geometry>
+        </visual>
+    </link>
+    <joint name ="rgb_camera_joint" type="fixed">
+        <parent link="base_link"/>
+        <child link = "rgb_camera"/>
+        <origin xyz="0 0.45 0.2" rpy="0 -0.5 1.57"/>
+    </joint>
 </robot>

Commit message: Add simulate robot

File: src/armbot_description/urdf/armbot.urdf.xacro (robot description, xacro)
@@ -4,6 +4,17 @@
     <xacro:property name="effort" value="30.0"/>
     <xacro:property name="velocity" value="10.0"/>
+    <!-- Useful Macros -->
+    <xacro:macro name="default_inertial" params="mass">
+        <inertial>
+            <origin xyz="0 0 0" rpy="0 0 0"/>
+            <mass value="${mass}" />
+            <inertia ixx="1.0" ixy="0.0" ixz="0.0"
+                     iyy="1.0" iyz="0.0"
+                     izz="1.0" />
+        </inertial>
+    </xacro:macro>
     <link name="world"/>
     <link name="base_link">
+        <xacro:default_inertial mass="1.0"/>
         <visual>
             <origin rpy="0 0 0" xyz="-0.5 -0.5 0"/>
@@ -25,4 +36,5 @@
     </joint>
     <link name="base_plate">
+        <xacro:default_inertial mass="0.1"/>
         <visual>
             <origin rpy="0 0 0" xyz="-0.39 -0.39 -0.56"/>
@@ -46,4 +58,5 @@
     </joint>
     <link name="forward_drive_arm">
+        <xacro:default_inertial mass="0.1"/>
         <visual>
             <origin rpy=" 0 -${PI / 2} ${PI / 2}" xyz="0.19 0.06 -0.08"/>
@@ -68,4 +81,5 @@
     </joint>
     <link name="horizontal_arm">
+        <xacro:default_inertial mass="0.1"/>
         <visual>
             <origin rpy="${PI / 2} 0 ${PI / 2}" xyz="-0.03 -0.4 -0.06"/>
@@ -90,4 +104,5 @@
     </joint>
     <link name="claw_support">
+        <xacro:default_inertial mass="0.05"/>
         <visual>
             <origin rpy="0 0 ${PI / 2}" xyz="0 -0.05 -0.15"/>
@@ -109,4 +124,5 @@
     </joint>
     <link name="gripper_right">
+        <xacro:default_inertial mass="0.01"/>
         <visual>
             <origin rpy="0 0 -${PI / 2}" xyz="-0.1 0.50 -0.1"/>
@@ -115,4 +131,10 @@
             </geometry>
         </visual>
+        <collision>
+            <origin rpy="0 0 -${PI / 2}" xyz="-0.1 0.50 -0.1"/>
+            <geometry>
+                <mesh filename="package://armbot_description/meshes/right_finger.STL" scale="0.01 0.01 0.01"/>
+            </geometry>
+        </collision>
     </link>
     <joint name ="joint_4" type="revolute">
@@ -125,4 +147,5 @@
     </joint>
     <link name="gripper_left">
+        <xacro:default_inertial mass="0.01"/>
         <visual>
             <origin rpy="0 0 -${PI / 2}" xyz="-0.04 0.50 -0.1"/>
@@ -131,4 +154,10 @@
             </geometry>
         </visual>
+        <collision>
+            <origin rpy="0 0 -${PI / 2}" xyz="-0.04 0.50 -0.1"/>
+            <geometry>
+                <mesh filename="package://armbot_description/meshes/left_finger.STL" scale="0.01 0.01 0.01"/>
+            </geometry>
+        </collision>
     </link>
     <joint name ="joint_5" type="revolute">
@@ -148,4 +177,10 @@
             </geometry>
         </visual>
+        <collision>
+            <origin rpy="-1.57 0 -1.57" xyz="-0.1 0.125 0.15"/>
+            <geometry>
+                <mesh filename="package://armbot_description/meshes/pi_camera.STL" scale="0.01 0.01 0.01"/>
+            </geometry>
+        </collision>
     </link>
     <joint name ="rgb_camera_joint" type="fixed">

Commit message: ROS2 control with gazebo

File: src/armbot_description/urdf/armbot.urdf.xacro (robot description, xacro)
@@ -1,4 +1,8 @@
 <?xml version="1.0"?>
 <robot xmlns:xacro="http://www.ros.org/wiki/xacro" name="armbot">
+    <!-- Include Gazebo Parameters -->
+    <xacro:include filename="$(find armbot_description)/urdf/armbot_gazebo.xacro" />
+    <!-- Include ros2_control Plugins -->
+    <xacro:include filename="$(find armbot_description)/urdf/armbot_ros2_control.xacro" />
     <xacro:property name="PI" value="3.14159"/>
     <xacro:property name="effort" value="30.0"/>
@@ -14,4 +18,13 @@
         </inertial>
     </xacro:macro>
+    <xacro:macro name="default_transmission" params="number">
+        <transmission name="transmission_${number}">
+            <plugin>transmission_interface/SimpleTransmission</plugin>
+            <actuator name="motor_${number}" role="actuator1"/>
+            <joint name="joint_${number}"    role="joint1">
+                <mechanical_reduction>1.0</mechanical_reduction>
+            </joint>
+        </transmission>
+    </xacro:macro>
     <link name="world"/>
     <link name="base_link">
@@ -190,35 +203,8 @@
         <origin xyz="0 0.45 0.2" rpy="0 -0.5 1.57"/>
     </joint>
-    <gazebo reference="rgb_camera">
-        <sensor type="camera" name="rgb_camera">
-            <always_on>true</always_on>
-            <update_rate>30.0</update_rate>
-            <camera name="rgb_camera">
-                <horizontal_fov>1.15</horizontal_fov>
-                <vertical_fov>0.71</vertical_fov>
-                <image>
-                    <width>2304</width>
-                    <height>1296</height>
-                    <format>R8G8B8</format>
-                </image>
-                <distortion>
-                    <k1>0.0</k1>
-                    <k2>0.0</k2>
-                    <k3>0.0</k3>
-                    <p1>0.0</p1>
-                    <p2>0.0</p2>
-                    <center>0.5 0.5</center>
-                </distortion>
-            </camera>
-            <plugin name="camera_controller" filename="libgazebo_ros_camera.so">
-                <ros>
-                    <remapping>~/image_raw:=image_raw</remapping>
-                    <remapping>~/camera_info:=camera_info</remapping>
-                </ros>
-                <camera_name>rgb_camera</camera_name>
-                <frame_name>rgb_camera</frame_name>
-                <hack_baseline>0.2</hack_baseline>
-            </plugin>
-        </sensor>
-    </gazebo>
+    <!-- Transmissions-->
+    <xacro:default_transmission number="1"/>
+    <xacro:default_transmission number="2"/>
+    <xacro:default_transmission number="3"/>
+    <xacro:default_transmission number="4"/>
 </robot>

File: src/armbot_description/urdf/armbot_gazebo.xacro (robot description, xacro)
@@ -33,3 +33,10 @@
         </sensor>
     </gazebo>
+    <gazebo>
+        <plugin filename="libgazebo_ros2_control.so" name="gazebo_ros2_control">
+            <robot_param>robot description</robot_param>
+            <robot_param_node>robot_state_publisher</robot_param_node>
+            <parameters/>
+        </plugin>
+    </gazebo>
 </robot>
